File: hw/electrical/line_sensor_encoder/line_sensor_encoder.kicad_pcb (KiCad board)
At the start: 2 copper layers, 45 x 66 mm, 45 parts, among them J1 Conn_02x04_Odd_Even, J2 Conn_02x06_Odd_Even, U1 TCRT5000L, U2 LM393, U3 TCRT5000L, U4 TCRT5000L, U5 TCRT5000L, U6 LM393, U7 TCRT5000L, U8 LM393

Commit message: added 3.3V dc converter
Parts:
- added C4: 22uF/10V, Capacitor_SMD:C_0805_2012Metric_Pad1.18x1.45mm_HandSolder, B.Cu at (130.8, 105.2)
- added C5: 22uF/10V, Capacitor_SMD:C_0805_2012Metric_Pad1.18x1.45mm_HandSolder, B.Cu at (130.7, 120.0)
- added U9: AMS1117-3.3, Package_TO_SOT_SMD:SOT-223-3_TabPin2, B.Cu at (131.0, 111.3)
- moved RV4 31.6 mm to (137.8, 106.7)
- moved RV5 31.6 mm to (137.8, 119.7)
- moved C1 31.6 mm to (150.2, 78.2)
- moved C2 31.6 mm to (150.8, 92.8)
- moved C3 31.6 mm to (150.8, 108.8)
- moved D1 31.6 mm to (143.5, 70.5)
- moved D2 31.6 mm to (143.5, 82.8)
- moved D3 31.6 mm to (143.5, 96.2)
- moved D4 31.6 mm to (143.5, 109.2)
- moved D5 31.6 mm to (143.5, 122.2)
- moved H1 31.6 mm to (150.8, 70.2)
- moved H2 31.6 mm to (150.8, 122.2)
- moved J1 31.6 mm to (131.5, 67.2)
- moved J2 31.6 mm to (131.5, 80.0)
- moved R1 31.6 mm to (167.2, 73.0)
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Connections:
- C1 pad 2: +5V -> +3.3V
- C2 pad 2: +5V -> +3.3V
- C3 pad 2: +5V -> +3.3V
- D1 pad 2: +5V -> +3.3V
- D2 pad 2: +5V -> +3.3V
- D3 pad 2: +5V -> +3.3V
- D4 pad 2: +5V -> +3.3V
- D5 pad 2: +5V -> +3.3V
- J2 pad 1: +5V -> +3.3V
- R1 pad 1: +5V -> +3.3V
- R10 pad 1: +5V -> +3.3V
- R11 pad 1: +5V -> +3.3V
- R12 pad 1: +5V -> +3.3V
- R13 pad 1: +5V -> +3.3V
- R14 pad 1: +5V -> +3.3V
- R17 pad 1: +5V -> +3.3V
- R18 pad 1: +5V -> +3.3V
- R19 pad 1: +5V -> +3.3V
- R2 pad 1: +5V -> +3.3V
- R3 pad 1: +5V -> +3.3V
- R4 pad 1: +5V -> +3.3V
- R5 pad 1: +5V -> +3.3V
- R7 pad 1: +5V -> +3.3V
- R9 pad 1: +5V -> +3.3V
- RV1 pad 1: +5V -> +3.3V
- RV2 pad 1: +5V -> +3.3V
- RV3 pad 1: +5V -> +3.3V
- RV4 pad 1: +5V -> +3.3V
- RV5 pad 1: +5V -> +3.3V
- U2 pad 8: +5V -> +3.3V
- U6 pad 8: +5V -> +3.3V
- U8 pad 8: +5V -> +3.3V
Routing:
- net +3.3V: track 0.00 -> 266.9 mm, vias 0 -> 2
- net +5V: track 314.0 -> 49.0 mm, vias 2 -> 0
- net /D5: track 79.6 -> 76.0 mm
Other:
- board text added: "5V"
- board text added: "Encoder v1.1"
- board text removed: "Line sensor encoder v1.0"
