File: hw/electrical/line_sensor_encoder/line_sensor_encoder.kicad_sch (KiCad schematic)
At the start: 45 parts, among them J1 Conn_02x04_Odd_Even, J2 Conn_02x06_Odd_Even, U1 TCRT5000L, U2 LM393, U3 TCRT5000L, U4 TCRT5000L, U5 TCRT5000L, U6 LM393, U7 TCRT5000L, U8 LM393

Commit message: added 3.3V dc converter
Parts:
- added C4, C5: 22uF/10V, Capacitor_SMD:C_0805_2012Metric_Pad1.18x1.45mm_HandSolder, symbol Device:C
- added U9: AMS1117-3.3, Package_TO_SOT_SMD:SOT-223-3_TabPin2, symbol Regulator_Linear:AMS1117-3.3
- U1, U3, U4, U5, U7: Availability (none) -> In Stock; Check_prices (none) -> https://www.snapeda.com/parts/TCRT5000L/Vishay+Semiconducto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; Package (none) -> PCB Mount Vishay; Price (none) -> None; Purchase-URL (none) -> https://www.snapeda.com/api/url_track_click_mouser/?unipart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; SnapEDA_Link (none) -> https://www.snapeda.com/parts/TCRT5000L/Vishay+Semiconducto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
Connections:
- net +5V: now also C4.1, U9.3 (VI); no longer C1.2, C2.2, C3.2, D1.2 (A), D2.2 (A), D3.2 (A), D4.2 (A), D5.2 (A), J2.1 (Pin_1), R1.1, R10.1, R11.1, R12.1, R13.1, R14.1, R17.1, R18.1, R19.1, R2.1, R3.1, R4.1, R5.1, R7.1, R9.1, RV1.1, RV2.1, RV3.1, RV4.1, RV5.1, U2.8 (V+), U6.8 (V+), U8.8 (V+)
- net GND: now also C4.2, C5.2, U9.1 (GND)
- new net +3.3V: C1.2, C2.2, C3.2, C5.1, D1.2 (A), D2.2 (A), D3.2 (A), D4.2 (A), D5.2 (A), J2.1 (Pin_1), R1.1, R10.1, R11.1, R12.1, R13.1, R14.1, R17.1, R18.1, R19.1, R2.1, R3.1, R4.1, R5.1, R7.1, R9.1, RV1.1, RV2.1, RV3.1, RV4.1, RV5.1, U2.8 (V+), U6.8 (V+), U8.8 (V+), U9.2 (VO)
Other:
- note added: "Voltage converter:"
- moved on the sheet: J1, J2

Commit message: added title block
Other:
- title: (none) -> Line sensor encoder
Changed lines of the file:
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@@
 (kicad_sch (version 20211123) (generator eeschema)
   (paper "A4")
+  (title_block
+    (title "Line sensor encoder")
+    (date "2023-09-02")
+    (rev "v.1.1")
+  )
   (junction (at 60.96 38.1) (diameter 0) (color 0 0 0 0)
   )
